File: Hardware/uCopter.brd (EAGLE design)
At the start: 50 x 50 mm, 50 parts, among them IC1 REG1117, IC2 STM32F303CBT, U1 MPU-6050, Y1 8M

Commit message: VERALTETE HARDWARE DIE NIE FUNKTIONIEREN WIRD!! NUR FÜR FREDERKIK!!!!! BITTESCHÖN \o\ \o/ /o/
Parts:
- added C13, C14: (no value), rcl:C0402
- added T1: BMP280, BOSCH-Testbuilds:BMP280
Connections:
- new net BMP_CSB: T1.P2
- new net BMP_SDO: T1.P5
- net +3,3V: now also C13.2, C14.2, T1.P6, T1.P8
- net GND: now also C13.1, C14.1, T1.P1, T1.P7
- net SCL: now also T1.P4
- net SDA: now also T1.P3
Routing:
- net +3,3V: track 75.8 -> 87.4 mm, vias 5 -> 6
- net GND: track 24.2 -> 26.2 mm, vias 53 -> 54
Changed lines of the file:
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@@
 <element name="R8" library="rcl" package="R0402" value="100k" x="11.875" y="33.625" rot="MR0"/>
 <element name="R10" library="rcl" package="R0402" value="100k" x="16.125" y="12" rot="MR270"/>
+<element name="T1" library="BOSCH-Testbuilds" package="BMP280" value="BMP280" x="35.875" y="30.5" rot="MR90"/>
+<element name="C13" library="rcl" package="C0402" value="" x="37.5" y="30.625" rot="MR90"/>
+<element name="C14" library="rcl" package="C0402" value="" x="35.5" y="32.375" rot="MR0"/>
 </elements>
 <signals>
@@
 <contactref element="C11" pad="2"/>
 <via x="23" y="23" extent="1-16" drill="0.35"/>
-<wire x1="29.25" y1="31.25" x2="28.375" y2="31.25" width="0.254" layer="1"/>
 <via x="19.625" y="27.375" extent="1-16" drill="0.35"/>
-<via x="25.375" y="31.25" extent="1-16" drill="0.35"/>
+<via x="25.5" y="31.375" extent="1-16" drill="0.35"/>
 <via x="16.375" y="28.75" extent="1-16" drill="0.35"/>
+<wire x1="28.5" y1="31.25" x2="28.375" y2="31.25" width="0.254" layer="1"/>
 <wire x1="20.75" y1="26.75" x2="20" y2="26.75" width="0.254" layer="1"/>
 <wire x1="20" y1="26.75" x2="19.75" y2="27" width="0.254" layer="1"/>
@@
 <wire x1="29.25" y1="31.25" x2="28.5" y2="31.25" width="0.254" layer="1"/>
 <wire x1="28.5" y1="31.25" x2="28.125" y2="30.875" width="0.254" layer="1"/>
-<via x="35.375" y="28.625" extent="1-16" drill="0.35"/>
+<via x="36.375" y="27.75" extent="1-16" drill="0.35"/>
 <via x="30.75" y="33.125" extent="1-16" drill="0.35"/>
-<via x="31.625" y="33.125" extent="1-16" drill="0.35"/>
+<via x="32.625" y="33" extent="1-16" drill="0.35"/>
 <via x="30.75" y="34" extent="1-16" drill="0.35"/>
 <via x="36.5" y="16.75" extent="1-16" drill="0.35"/>
@@
 <via x="35.375" y="27.75" extent="1-16" drill="0.35"/>
 <via x="35.375" y="26.875" extent="1-16" drill="0.35"/>
-<via x="26.9375" y="30.875" extent="1-16" drill="0.35"/>
 <wire x1="28.125" y1="30.875" x2="27.875" y2="30.875" width="0.254" layer="1"/>
-<via x="36.25" y="32.25" extent="1-16" drill="0.35"/>
-<via x="35.375" y="32.25" extent="1-16" drill="0.35"/>
-<via x="34.5" y="32.25" extent="1-16" drill="0.35"/>
+<via x="34.5" y="34.625" extent="1-16" drill="0.35"/>
+<via x="35.375" y="33.75" extent="1-16" drill="0.35"/>
+<via x="34.5" y="33.75" extent="1-16" drill="0.35"/>
 <via x="19.39" y="32.205" extent="1-16" drill="0.35"/>
 <via x="21.375" y="25.125" extent="1-16" drill="0.35"/>
@@
 <wire x1="23.03125" y1="32.28125" x2="23.03125" y2="31.78125" width="0.254" layer="1"/>
 <wire x1="23.03125" y1="31.78125" x2="23" y2="31.375" width="0.254" layer="1"/>
-<wire x1="22.75" y1="34.375" x2="20.625" y2="34.375" width="0.254" layer="1"/>
 <wire x1="20.625" y1="34.375" x2="20" y2="33.75" width="0.4064" layer="1"/>
 <wire x1="20" y1="33.75" x2="20" y2="33.275" width="0.4064" layer="1"/>
@@
 <wire x1="29.25" y1="31.25" x2="30" y2="31.25" width="0.3048" layer="1"/>
 <wire x1="30" y1="31.25" x2="30.375" y2="31.625" width="0.3048" layer="1"/>
-<wire x1="30.375" y1="31.625" x2="30.375" y2="32.75" width="0.3048" layer="1"/>
-<wire x1="30.375" y1="32.75" x2="30.75" y2="33.125" width="0.3048" layer="1"/>
 <wire x1="25.75" y1="24.75" x2="25.75" y2="25.5" width="0.3048" layer="1"/>
 <wire x1="25.75" y1="25.5" x2="25.5" y2="25.75" width="0.3048" layer="1"/>
-<wire x1="23" y1="31.375" x2="25.375" y2="31.25" width="0" layer="19" extent="1-1"/>
-<wire x1="27" y1="26.25" x2="25.75" y2="25.5" width="0" layer="19" extent="1-16"/>
+<wire x1="27" y1="26.25" x2="24.375" y2="26.25" width="0.254" layer="16"/>
+<wire x1="24.375" y1="26.25" x2="24.125" y2="26" width="0.254" layer="16"/>
+<via x="24.125" y="26" extent="1-16" drill="0.35"/>
+<wire x1="24.125" y1="26" x2="25.25" y2="26" width="0.254" layer="1"/>
+<wire x1="25.25" y1="26" x2="25.75" y2="25.5" width="0.254" layer="1"/>
+<contactref element="T1" pad="P1"/>
+<contactref element="T1" pad="P7"/>
+<wire x1="36.375" y1="30" x2="36.375" y2="29.625" width="0.254" layer="16"/>
+<contactref element="C13" pad="1"/>
+<contactref element="C14" pad="1"/>
+<wire x1="36.375" y1="30" x2="36.375" y2="30.25" width="0.254" layer="16"/>
+<wire x1="36.375" y1="30.25" x2="35.875" y2="30.75" width="0.254" layer="16"/>
+<wire x1="35.875" y1="30.75" x2="35.875" y2="31" width="0.254" layer="16"/>
+<via x="30.375" y="31.75" extent="1-16" drill="0.35"/>
+<wire x1="30.375" y1="31.75" x2="30.375" y2="31.625" width="0.254" layer="1"/>
 </signal>
 <signal name="N$1">
@@
 <wire x1="21.125" y1="23.125" x2="21.65" y2="23.65" width="0.254" layer="16"/>
 <wire x1="21.65" y1="23.65" x2="22" y2="23.65" width="0.254" layer="16"/>
+<contactref element="T1" pad="P6"/>
+<contactref element="T1" pad="P8"/>
+<contactref element="C13" pad="2"/>
+<contactref element="C14" pad="2"/>
+<wire x1="36.375" y1="31" x2="37.5" y2="31" width="0.254" layer="16"/>
+<wire x1="37.5" y1="31" x2="37.5" y2="31.275" width="0.254" layer="16"/>
+<wire x1="34.85" y1="32.375" x2="35.375" y2="31.85" width="0.254" layer="16"/>
+<wire x1="35.375" y1="31.85" x2="35.375" y2="31" width="0.254" layer="16"/>
+<wire x1="36.375" y1="31" x2="36.375" y2="31.375" width="0.254" layer="16"/>
+<wire x1="36.375" y1="31.375" x2="36.125" y2="31.625" width="0.254" layer="16"/>
+<wire x1="36.125" y1="31.625" x2="35.6" y2="31.625" width="0.254" layer="16"/>
+<wire x1="35.6" y1="31.625" x2="35.375" y2="31.85" width="0.254" layer="16"/>
+<wire x1="34.85" y1="32.375" x2="34.25" y2="32.375" width="0.254" layer="16"/>
+<via x="32.625" y="34" extent="1-16" drill="0.35"/>
+<wire x1="32.625" y1="34" x2="31" y2="32.375" width="0.254" layer="1"/>
+<wire x1="31" y1="32.375" x2="29.475" y2="32.375" width="0.254" layer="1"/>
+<wire x1="29.475" y1="32.375" x2="29.25" y2="32.6" width="0.254" layer="1"/>
+<wire x1="32.625" y1="34" x2="34.25" y2="32.375" width="0.254" layer="16"/>
 </signal>
 <signal name="SCL">
@@
 <wire x1="21.75" y1="31" x2="21.5" y2="31.25" width="0.254" layer="1"/>
 <wire x1="21.5" y1="31.25" x2="20.75" y2="31.25" width="0.254" layer="1"/>
+<contactref element="T1" pad="P4"/>
+<wire x1="25.9375" y1="28.1" x2="34.875" y2="30" width="0" layer="19" extent="16-16"/>
 </signal>
 <signal name="SDA">
@@
 <wire x1="22.25" y1="31.125" x2="21.625" y2="31.75" width="0.254" layer="1"/>
 <wire x1="21.625" y1="31.75" x2="20.75" y2="31.75" width="0.254" layer="1"/>
+<contactref element="T1" pad="P3"/>
+<wire x1="27" y1="28.5" x2="35.375" y2="30" width="0" layer="19" extent="16-16"/>
 </signal>
 <signal name="N$7">
@@
 <wire x1="22.125" y1="28.375" x2="25.5" y2="28.375" width="0.254" layer="1"/>
 <wire x1="25.5" y1="28.375" x2="25.75" y2="28.625" width="0.254" layer="1"/>
-<wire x1="25.75" y1="28.625" x2="25.75" y2="29.875" width="0.254" layer="1"/>
-<wire x1="25.75" y1="29.875" x2="24.375" y2="31.25" width="0.254" layer="1"/>
-<via x="24.375" y="31.25" extent="1-16" drill="0.35"/>
-<wire x1="24.375" y1="31.25" x2="24.375" y2="31.75" width="0.254" layer="16"/>
+<wire x1="25.75" y1="28.625" x2="25.75" y2="30" width="0.254" layer="1"/>
+<wire x1="25.75" y1="30" x2="24.375" y2="31.375" width="0.254" layer="1"/>
+<via x="24.375" y="31.375" extent="1-16" drill="0.35"/>
+<wire x1="24.375" y1="31.375" x2="24.375" y2="31.75" width="0.254" layer="16"/>
 <wire x1="24.375" y1="31.75" x2="25" y2="32.375" width="0.254" layer="16"/>
 <wire x1="25" y1="32.375" x2="33.5" y2="32.375" width="0.254" layer="16"/>
@@
 <wire x1="14.625" y1="15.875" x2="14.625" y2="32.375" width="0.254" layer="16"/>
 <wire x1="14.625" y1="32.375" x2="16.625" y2="34.375" width="0.254" layer="16"/>
-<wire x1="16.625" y1="34.375" x2="21" y2="34.375" width="0.254" layer="16"/>
-<wire x1="21" y1="34.375" x2="21.125" y2="34.25" width="0.254" layer="16"/>
-<wire x1="21.125" y1="34.25" x2="21.875" y2="34.25" width="0.254" layer="16"/>
-<wire x1="21.875" y1="34.25" x2="22" y2="34.375" width="0.254" layer="16"/>
-<wire x1="22" y1="34.375" x2="24.75" y2="34.375" width="0.254" layer="16"/>
+<wire x1="16.625" y1="34.375" x2="20.875" y2="34.375" width="0.254" layer="16"/>
+<wire x1="20.875" y1="34.375" x2="21" y2="34.25" width="0.254" layer="16"/>
+<wire x1="21" y1="34.25" x2="22" y2="34.25" width="0.254" layer="16"/>
+<wire x1="22" y1="34.25" x2="22.125" y2="34.375" width="0.254" layer="16"/>
+<wire x1="22.125" y1="34.375" x2="24.75" y2="34.375" width="0.254" layer="16"/>
 <via x="24.75" y="34.375" extent="1-16" drill="0.35"/>
 <wire x1="24.75" y1="34.375" x2="24.75" y2="33.25" width="0.254" layer="1"/>
@@
 <wire x1="24.25" y1="32.25" x2="24.25" y2="33.25" width="0.254" layer="1"/>
 </signal>
+<signal name="BMP_CSB">
+<contactref element="T1" pad="P2"/>
+</signal>
+<signal name="BMP_SDO">
+<contactref element="T1" pad="P5"/>
+</signal>
 </signals>
